Commit message: Update ur10_robot_stick.urdf
longer stick

File: ur_description/urdf/ur10_robot_stick.urdf (robot description, URDF)
Before this commit: robot ur10, 13 links, 12 joints
Links:
- link stick: geometry collision mesh filename=package://ur_description/meshes/ur10/collision/stick.stl scale=0.001 0.001 0.00245; visual mesh filename=package://ur_description/meshes/ur10/visual/stick.obj scale=0.001 0.001 0.00245
